File: magnetic_levitator_mcu.kicad_pcb (KiCad board)
At the start: 2 copper layers, 62 x 25 mm, 33 parts, among them J1 USB_C_Receptacle_USB2.0, J2 Conn_01x03, J3 Conn_01x03, J4 Conn_01x04, J5 Conn_01x02, J6 Conn_01x02, J7 Barrel_Jack_Switch, Q1 BSC0702LS, U1 STM32C011F6Px, U3 UCC27511ADBV, U4 HT75xx-1-SOT89

Commit message: WIP
Parts:
- removed H1, H2, H3, H4: MountingHole, MountingHole:MountingHole_2.2mm_M2
- removed J2, J3: Conn_01x03, Connector_PinHeader_2.54mm:PinHeader_1x03_P2.54mm_Vertical
- added C11: 100nF, Capacitor_SMD:C_0402_1005Metric, F.Cu at (97.2, 99.2)
- added C12: 1nF, Capacitor_SMD:C_0402_1005Metric, F.Cu at (97.2, 101.2)
- added C13: 10nF, Capacitor_SMD:C_0402_1005Metric, F.Cu at (97.2, 103.2)
- added C14: 100nF, Capacitor_SMD:C_0402_1005Metric, F.Cu at (97.2, 105.1)
- added Q2: MMBT2222A, Package_TO_SOT_SMD:SOT-23, F.Cu at (101.1, 100.6)
- added R29: 220k, Resistor_SMD:R_0603_1608Metric, F.Cu at (100.6, 104.1)
- added R30: 5.1k, Resistor_SMD:R_0402_1005Metric, F.Cu at (94.3, 99.2)
- added R31: 47, Resistor_SMD:R_0402_1005Metric, F.Cu at (94.3, 101.2)
- added R32: 47, Resistor_SMD:R_0402_1005Metric, F.Cu at (94.3, 103.2)
- added R33: 5.1k, Resistor_SMD:R_0402_1005Metric, F.Cu at (94.3, 105.2)
- added R34: 5.1k, Resistor_SMD:R_0402_1005Metric, F.Cu at (94.3, 107.2)
- added U2: LM358, Package_SO:SOIC-8_3.9x4.9mm_P1.27mm, F.Cu at (133.9, 118.8)
- added U5: ~, gabe_sensors:TCRT1000, F.Cu at (110.8, 102.0)
- U4: value HT75xx-1-SOT89 -> HT7533-1
Connections:
- U1 pad 6: unconnected-(U1-PF2-Pad6) -> Net-(U1-PF2)
- U1 pad 7: Net-(J2-Pin_2) -> /ADC
- U1 pad 8: Net-(J3-Pin_2) -> unconnected-(U1-PA1-Pad8)
